File: ambra.kicad_pcb (KiCad board)
At the start: 2 copper layers, 148.6 x 86.3 mm, 34 parts, among them J1 MJ-4PP-9, SW1 SW_SPDT, U1 ProMicro_r

Commit message: Add files via upload
Parts:
- removed the REF** at (92.4, 120.3)
- removed the REF** at (171.9, 120.3)
- added REF**: RTLECS MG03254 90 m, my syms-foots:RTLECS_MG03254_90_m, B.Cu at (172.0, 120.3)
- added REF**: RTLECS_MG03254_f, my syms-foots:RTLECS_MG03254_f, B.Cu at (92.3, 120.3)
- moved BT3 13.9 mm to (100.1, 111.5)
- moved ? 2.88 mm to (165.2, 124.3)
- moved ? 2.88 mm to (99.6, 123.5)
- moved ? 2.85 mm to (87.8, 126.7)
- moved ? 2.85 mm to (169.3, 112.8)
Routing:
- net Net-(SW1-C): track 44.2 -> 36.2 mm
- net reset: track 48.7 -> 40.8 mm
- net VBAT: track 59.4 -> 53.3 mm
Other:
- outline, holes or cut-outs redrawn

Commit message: Add files via upload
Parts:
- removed the ? at (99.6, 123.5)
- removed the ? at (87.8, 126.7)
- removed the BT3 at (94.4, 90.2)
- removed the SWr1c5 at (84.9, 92.1)
- removed the SWr2c5 at (89.3, 108.5)
- added BT3: Breakaway Tabs, kbd_local:Breakaway_Tabs, F.Cu at (157.4, 127.9)
- added BT3: Breakaway Tabs, kbd_local:Breakaway_Tabs, F.Cu at (158.6, 125.7)
- added H1: Hole, enki_lib:HOLE, F.Cu at (143.4, 122.9)
- added SWr4c1: SW_PUSH, my syms-foots:ChocV1_duplex_hotswap_topor, F.Cu at (149.1, 134.3)
- added SWr4c2: SW_PUSH, enki_lib:ChocV1_duplex_hotswap_topor, F.Cu at (131.3, 126.1)
- moved REF** 68.6 mm to (158.1, 139.7), turned to 60 degrees
- moved BT3 32.4 mm to (132.2, 116.1), turned to -20 degrees
Routing:
- net GND2: track 68.5 -> 0.00 mm
- net db2: track 30.7 -> 0.00 mm
- net db1: track 30.6 -> 0.00 mm
- net VCC: track 46.0 -> 42.1 mm
Other:
- board size 148.6 x 86.3 mm -> 129.9 x 99.4 mm
- board text removed: "<-board"
- board text removed: "board->"

Commit message: Add files via upload
Other:
- board size 129.9 x 99.4 mm -> 129.8 x 99.4 mm
Changed lines of the file:
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@@
 		)
 	)
-	(footprint ""
-		(layer "F.Cu")
-		(at 169.33 112.83)
-		(property "Reference" ""
-			(at 0 0 0)
-			(layer "F.SilkS")
-			(effects
-				(font
-					(size 1.27 1.27)
-					(thickness 0.15)
-				)
-			)
-		)
-		(property "Value" ""
-			(at 0 0 0)
-			(layer "F.Fab")
-			(effects
-				(font
-					(size 1.27 1.27)
-					(thickness 0.15)
-				)
-			)
-		)
-		(property "Footprint" ""
-			(at 0 0 0)
-			(layer "F.Fab")
-			(hide yes)
-			(effects
-				(font
-					(size 1.27 1.27)
-					(thickness 0.15)
-				)
-			)
-		)
-		(property "Datasheet" ""
-			(at 0 0 0)
-			(layer "F.Fab")
-			(hide yes)
-			(effects
-				(font
-					(size 1.27 1.27)
-					(thickness 0.15)
-				)
-			)
-		)
-		(property "Description" ""
-			(at 0 0 0)
-			(layer "F.Fab")
-			(hide yes)
-			(effects
-				(font
-					(size 1.27 1.27)
-					(thickness 0.15)
-				)
-			)
-		)
-		(pad "1" thru_hole circle
-			(at 0 0 355)
-			(size 4.4 4.4)
-			(drill 2.2)
-			(layers "*.Cu" "*.Mask")
-			(remove_unused_layers no)
-		)
-	)
 	(footprint "enki_lib:ChocV1_duplex_hotswap_topor"
 		(layer "F.Cu")
@@
 		(at 165.15 124.29)
 		(property "Reference" ""
-			(at -3.642154 -1.328469 0)
+			(at 0 0 0)
 			(layer "F.SilkS")
 			(effects
@@
 		)
 		(property "Value" ""
-			(at -3.642154 -1.328469 0)
+			(at 0 0 0)
 			(layer "F.Fab")
 			(effects
@@
 			)
 		)
-		(pad "1" thru_hole circle
-			(at 0 0 355)
-			(size 4.4 4.4)
-			(drill 2.2)
+		(pad "" np_thru_hole circle
+			(at 0 0)
+			(size 2.4 2.4)
+			(drill 2.1)
 			(layers "*.Cu" "*.Mask")
-			(remove_unused_layers no)
 		)
 	)
@@
 		)
 	)
+	(footprint ""
+		(layer "F.Cu")
+		(at 169.33 112.83)
+		(property "Reference" ""
+			(at 0 0 0)
+			(layer "F.SilkS")
+			(effects
+				(font
+					(size 1.27 1.27)
+					(thickness 0.15)
+				)
+			)
+		)
+		(property "Value" ""
+			(at 0 0 0)
+			(layer "F.Fab")
+			(effects
+				(font
+					(size 1.27 1.27)
+					(thickness 0.15)
+				)
+			)
+		)
+		(property "Footprint" ""
+			(at 0 0 0)
+			(layer "F.Fab")
+			(hide yes)
+			(effects
+				(font
+					(size 1.27 1.27)
+					(thickness 0.15)
+				)
+			)
+		)
+		(property "Datasheet" ""
+			(at 0 0 0)
+			(layer "F.Fab")
+			(hide yes)
+			(effects
+				(font
+					(size 1.27 1.27)
+					(thickness 0.15)
+				)
+			)
+		)
+		(property "Description" ""
+			(at 0 0 0)
+			(layer "F.Fab")
+			(hide yes)
+			(effects
+				(font
+					(size 1.27 1.27)
+					(thickness 0.15)
+				)
+			)
+		)
+		(pad "" np_thru_hole circle
+			(at 0 0)
+			(size 2.4 2.4)
+			(drill 2.1)
+			(layers "*.Cu" "*.Mask")
+		)
+	)
 	(footprint "kbd_local:Breakaway_Tabs"
 		(layer "F.Cu")
@@
 	)
 	(gr_line
-		(start 144.707288 120.86995)
+		(start 144.747288 120.88995)
 		(end 155.2 126.92)
 		(stroke
@@
 	(gr_line
 		(start 155.2 126.92)
-		(end 155.397205 126.58801)
+		(end 155.42 126.54)
 		(stroke
 			(width 0.15)
@@
 	(gr_line
 		(start 143.638581 120.033893)
-		(end 156.46 124.71)
+		(end 156.41 124.69)
 		(stroke
 			(width 0.15)
@@
 	)
 	(gr_arc
-		(start 221.940024 78.819431)
-		(mid 222.618877 79.17288)
-		(end 222.849062 79.902781)
+		(start 221.927324 78.819431)
+		(mid 222.606136 79.172883)
+		(end 222.836362 79.902781)
 		(stroke
 			(width 0.15)
@@
 	)
 	(gr_line
-		(start 220.458375 95.754741)
+		(start 220.452875 95.756241)
 		(end 215.327972 95.305888)
 		(stroke
@@
 	)
 	(gr_line
-		(start 221.541726 94.845701)
-		(end 222.849062 79.902781)
+		(start 221.536225 94.847201)
+		(end 222.836362 79.902781)
 		(stroke
 			(width 0.15)
@@
 	)
 	(gr_line
-		(start 156.46 124.71)
-		(end 156.29 125.04)
+		(start 156.41 124.69)
+		(end 156.28 125.05)
 		(stroke
 			(width 0.15)
@@
 	(gr_line
 		(start 197.035155 76.640538)
-		(end 221.940022 78.81943)
+		(end 221.927324 78.819431)
 		(stroke
 			(width 0.15)
@@
 	)
 	(gr_arc
-		(start 221.541725 94.845701)
-		(mid 221.188313 95.524591)
-		(end 220.458375 95.754741)
+		(start 221.536225 94.847201)
+		(mid 221.182807 95.526073)
+		(end 220.452875 95.756241)
 		(stroke
 			(width 0.15)
@@
 	)
 	(gr_line
-		(start 156.29 125.04)
-		(end 155.397205 126.58801)
+		(start 156.28 125.05)
+		(end 155.42 126.54)
 		(stroke
 			(width 0.15)
@@
 	)
 	(gr_arc
-		(start 144.452846 120.751531)
-		(mid 144.615363 120.814519)
-		(end 144.767288 120.89995)
+		(start 144.432846 120.741531)
+		(mid 144.59536 120.804526)
+		(end 144.747288 120.88995)
 		(stroke
 			(width 0.15)
@@
 	(gr_line
 		(start 134.315441 117.055066)
-		(end 144.338509 120.707157)
+		(end 144.432846 120.741531)
 		(stroke
 			(width 0.15)
@@
 		(layer "Edge.Cuts")
 	)
-	(gr_line
-		(start 144.338509 120.707157)
-		(end 144.432846 120.741531)
-		(stroke
-			(width 0.15)
-			(type solid)
-		)
-		(layer "Edge.Cuts")
-	)
 	(gr_arc
 		(start 105.877718 128.988333)
@@
 	)
 	(gr_line
-		(start 221.533312 94.85385)
-		(end 222.840648 79.91093)
-		(stroke
-			(width 0.15)
-			(type solid)
-		)
-		(layer "Edge.Cuts")
-	)
-	(gr_line
 		(start 129.651561 115.355695)
 		(end 129.847427 115.427062)
@@
 		(stroke
 			(width 0.15)
-			(type solid)
-		)
-		(layer "Edge.Cuts")
-	)
-	(gr_arc
-		(start 221.93161 78.82758)
-		(mid 222.610451 79.181028)
-		(end 222.840648 79.91093)
-		(stroke
-			(width 0.15)

Commit message: Add files via upload
Parts:
- moved REF** 4.03 mm to (162.0, 140.5)
- moved BT3 3.97 mm to (162.4, 127.1)
- moved BT3 3.93 mm to (160.9, 129.7)
- moved SWr4c2 1.69 mm to (132.9, 125.6), turned to -20 degrees
- moved H1 1.69 mm to (145.0, 122.4)
- moved SWr4c1 1.69 mm to (150.7, 133.9), turned to -30 degrees
Other:
- outline, holes or cut-outs redrawn

Commit message: Add files via upload
Parts:
- removed the REF** at (206.4, 81.0)
- removed the REF** at (204.4, 80.9)
- added REF**: JST_B2B-ZR_LF__SN_, my syms-foots:JST_B2B-ZR_LF__SN_, F.Cu at (204.9, 82.6)
- added REF**: JST_B2B-ZR_LF__SN_, my syms-foots:JST_B2B-ZR_LF__SN_, B.Cu at (204.0, 81.5)
Routing:
- net VCC: track 42.1 -> 31.6 mm
- net GND: track 671.6 -> 667.8 mm

Commit message: Add files via upload
Parts:
- moved REF** 1.60 mm to (160.7, 139.7)
Other:
- board size 129.8 x 99.4 mm -> 129.8 x 98.6 mm

Commit message: Add files via upload
Parts:
- added P6SMBJ5.0CA: ZENER, Library:P6SMBJ5.0CA, F.Cu at (209.5, 80.2)
- added REF**: BEADC1608X95N, BLM18PG121SN1D:BEADC1608X95N, F.Cu at (217.3, 94.2)
- added REF**: BEADC1608X95N, BLM18PG121SN1D:BEADC1608X95N, B.Cu at (195.6, 84.2)
- added REF**: BEADC1608X95N, BLM18PG121SN1D:BEADC1608X95N, B.Cu at (214.1, 79.2)
- added REF**: BEADC1608X95N, BLM18PG121SN1D:BEADC1608X95N, B.Cu at (197.9, 78.0)
Routing:
- net r2c3: track 98.6 -> 78.6 mm
- net r1c1: track 95.6 -> 79.3 mm
- net r3c5: track 118.3 -> 105.4 mm
- net GND: track 667.8 -> 655.6 mm, vias 2 -> 13
- net r1c2: track 109.9 -> 102.6 mm
- net VCC: track 31.6 -> 27.4 mm, vias 1 -> 2
- added copper zone on B.Cu, net GND
- added copper zone on F.Cu, net GND
Other:
- outline, holes or cut-outs redrawn

Commit message: Add files via upload
Routing:
- net GND2: track 0.00 -> 75.1 mm
- net db2: track 0.00 -> 59.7 mm
- net db1: track 0.00 -> 40.3 mm
- net GND: track 655.6 -> 692.6 mm
- net reset: track 40.8 -> 60.8 mm
- net VCC: track 27.4 -> 44.2 mm
- net Net-(SW1-C): track 36.2 -> 47.3 mm
