File: ambra.kicad_pcb (KiCad board)
At the start: 2 copper layers, 129.8 x 98.6 mm, 39 parts, among them J1 MJ-4PP-9, P6SMBJ5.0CA ZENER, SW1 SW_SPDT, U1 ProMicro_r

Commit message: Add files via upload
Parts:
- removed P6SMBJ5.0CA: ZENER, Library:P6SMBJ5.0CA
- removed the REF** at (217.3, 94.2)
- removed the REF** at (204.9, 82.6)
- removed the REF** at (195.6, 84.2)
- removed the REF** at (214.1, 79.2)
- removed the REF** at (197.9, 78.0)
- removed the REF** at (204.0, 81.5)
- added REF**: JST_B2B-ZR_LF__SN_, my syms-foots:JST_B2B-ZR_LF__SN_, F.Cu at (204.4, 82.2)
- J1: footprint enki_lib:MJ-4PP-9_dual_topor -> my syms-foots:TRRS-MJ-4PP-9_dual_topor
- SWr1c1, SWr1c2, SWr1c3, SWr1c4, SWr2c1, SWr2c2, SWr2c3, SWr2c4, SWr3c1, SWr3c2, SWr3c3, SWr3c4, SWr3c5, SWr4c2: footprint enki_lib:ChocV1_duplex_hotswap_topor -> my syms-foots:ChocV1_duplex_hotswap_topor
- U1: footprint enki_lib:ProMicro_duplex_clean -> my syms-foots:ProMicro_duplex_clean
- moved ? 0.13 mm to (214.9, 94.1)
Connections:
- U1 pad 1: r3c3 -> r2c4
- U1 pad 10: r3c5 -> r3c3
- U1 pad 11: r4c2 -> r2c5
- U1 pad 12: r4c1 -> r3c5
- U1 pad 13: r3c1 -> r4c2
- U1 pad 14: r1c2 -> r4c1
- U1 pad 15: r2c2 -> r3c1
- U1 pad 16: r3c2 -> r1c5
- U1 pad 17: r1c3 -> r1c4
- U1 pad 18: r2c3 -> r1c3
- U1 pad 19: r2c1 -> r1c2
- U1 pad 2: r1c4 -> r2c1
- U1 pad 6: r2c4 -> r2c2
- U1 pad 7: r3c4 -> r2c3
- U1 pad 8: r1c5 -> r3c4
- U1 pad 9: r2c5 -> r3c2
Routing:
- net GND: track 692.6 -> 58.7 mm, vias 13 -> 18
- net Net-(SW1-C): track 47.3 -> 106.3 mm, vias 1 -> 0
- net VBAT: track 53.3 -> 110.4 mm, vias 2 -> 3
- net r1c5: track 145.4 -> 176.9 mm, vias 1 -> 2
- net r4c1: track 22.5 -> 50.6 mm
- net r3c5: track 105.4 -> 133.2 mm, vias 1 -> 2
- net reset: track 60.8 -> 86.0 mm, vias 3 -> 2
- net r4c2: track 26.6 -> 51.5 mm
- net r1c4: track 121.5 -> 145.1 mm, vias 1 -> 2
- net r2c5: track 108.6 -> 130.5 mm, vias 1 -> 2
- net r2c2: track 93.7 -> 72.3 mm
- net r2c3: track 78.6 -> 95.9 mm, vias 1 -> 2
- net VCC: track 44.2 -> 27.7 mm, vias 2 -> 1
- net r1c1: track 79.3 -> 74.3 mm, vias 1 -> 2
- net r3c1: track 55.5 -> 50.6 mm, vias 1 -> 2
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- removed copper zone on F.Cu, net GND
Other:
- board text added: "- +"
- board text removed: "- + -"
- board text removed: "dsn: tapioki, Aroum, stozi"

Commit message: Add files via upload
Routing:
- net r2c1: track 49.4 -> 50.9 mm
- net r1c1: track 74.3 -> 75.0 mm

Commit message: Add files via upload
Routing:
- net Net-(SW1-C): track 106.3 -> 104.9 mm
- net VBAT: track 110.4 -> 109.1 mm

Commit message: Add files via upload
Routing:
- net r1c3: track 121.3 -> 124.6 mm
- net r1c5: track 176.9 -> 180.1 mm
- net r3c3: track 95.4 -> 98.2 mm
- net r1c4: track 145.1 -> 147.3 mm
- net r3c1: track 50.6 -> 52.8 mm
- net r2c1: track 50.9 -> 52.0 mm
- net r3c4: track 119.7 -> 120.8 mm
- net Net-(SW1-C): track 104.9 -> 103.8 mm
- net r2c4: track 126.5 -> 127.4 mm
- net r1c2: track 98.2 -> 99.0 mm
- net reset: track 86.0 -> 85.4 mm
- net r3c2: track 74.0 -> 73.4 mm

Commit message: Add files via upload
Parts:
- RSW1: footprint enki_lib:SW_3x4x2_2legs_x2 -> my syms-foots:reset-SW_3x4x2_2legs_x2
- SW1: footprint enki_lib:switch_MSK-12C02_smd_x2_topor -> my syms-foots:switch_MSK-12C02_smd_x2_topor
- SWr1c5, SWr2c5: footprint enki_lib:ChocV1_duplex_hotswap_topor -> my syms-foots:ChocV1_duplex_hotswap_topor
Connections:
- U1 pad 1: r2c4 -> r2c3
- U1 pad 10: r3c3 -> r3c4
- U1 pad 16: r1c5 -> r2c4
- U1 pad 7: r2c3 -> r1c5
- U1 pad 8: r3c4 -> r3c3
Routing:
- net r1c5: track 180.1 -> 142.1 mm
- net r2c4: track 127.4 -> 159.1 mm
- net r3c4: track 120.8 -> 114.3 mm
- net r2c3: track 96.1 -> 101.4 mm
- net r3c3: track 98.2 -> 95.9 mm
- net r2c5: track 130.5 -> 129.7 mm
- net r1c2: track 99.0 -> 98.2 mm
- net r1c3: track 124.6 -> 123.9 mm

Commit message: Add files via upload
Connections:
- U1 pad 1: r2c3 -> r2c2
- U1 pad 16: r2c4 -> r2c3
- U1 pad 6: r2c2 -> r2c4
Routing:
- net r2c4: track 159.1 -> 119.5 mm
- net r2c3: track 101.4 -> 124.9 mm
- net r2c2: track 72.6 -> 76.3 mm
- net r1c1: track 75.0 -> 76.8 mm
- net r1c4: track 147.2 -> 146.5 mm

Commit message: Add files via upload
Parts:
- removed the REF** at (204.4, 82.2)
- added REF**: JST_B3B-PH-K-S, my syms-foots:JST-PH, F.Cu at (203.8, 83.8)
Connections:
- SW1 pad 2: VBAT -> VCC
- U1 pad 24: VBAT -> (no net)
- U1 pad B+: Net-(SW1-C) -> (no net)
Routing:
- net VBAT: track 108.6 -> 0.00 mm, vias 3 -> 0
- net VCC: track 27.7 -> 119.5 mm, vias 1 -> 3
- net Net-(SW1-C): track 103.8 -> 94.5 mm
- net r2c1: track 52.0 -> 59.2 mm
- net r2c3: track 124.9 -> 130.1 mm
- net r1c1: track 76.8 -> 80.5 mm
- net r2c2: track 76.3 -> 78.3 mm
- net r1c4: track 146.5 -> 145.4 mm
- net r4c2: track 51.8 -> 50.9 mm
- net GND: track 58.7 -> 59.6 mm, vias 18 -> 17
- net r1c2: track 98.2 -> 97.4 mm
- net reset: track 85.4 -> 86.1 mm
- net r1c3: track 123.9 -> 123.4 mm
Other:
- board text added: "+"
- board text removed: "- +"

Commit message: Add files via upload
Parts:
- added REF**: CAPC1608X95N, my syms-foots:CAPC1608X95N, B.Cu at (203.4, 91.1)
- added REF**: CAPC3225X270N, my syms-foots:CAPC3225X270N, B.Cu at (187.9, 111.9)
Routing:
- net GND: track 59.6 -> 57.8 mm
- net VCC: track 119.5 -> 119.8 mm, vias 3 -> 4
