File: ambra.kicad_pcb (KiCad board)
At the start: 2 copper layers, 129.8 x 98.6 mm, 33 parts, among them J1 MJ-4PP-9, SW1 SW_SPDT, U1 ProMicro_r

Commit message: Add files via upload
Routing:
- net r3c1: track 53.8 -> 51.9 mm

Commit message: Add files via upload
Routing:
- net r2c2: track 76.8 -> 75.8 mm

Commit message: Add files via upload
Routing:
- net r3c5: track 143.9 -> 143.2 mm

Commit message: Add files via upload
Routing:
- net r1c5: track 142.4 -> 138.3 mm
- net r3c1: track 51.9 -> 48.3 mm
- net r1c1: track 77.3 -> 73.8 mm
- net GND: track 61.9 -> 58.9 mm
- net r2c4: track 119.5 -> 116.6 mm
- net r3c2: track 72.4 -> 69.6 mm
- net r1c2: track 95.6 -> 92.9 mm
- net r2c1: track 53.8 -> 51.5 mm
- net r3c4: track 112.9 -> 111.3 mm
- net r1c4: track 144.2 -> 142.8 mm
- net r2c2: track 75.8 -> 74.9 mm
- net r3c5: track 143.2 -> 142.5 mm
- net VCC: track 27.6 -> 26.9 mm
- net r2c5: track 128.8 -> 128.0 mm
- net data: track 33.7 -> 33.1 mm

Commit message: Add files via upload
Parts:
- SWr1c1, SWr1c2, SWr1c3, SWr1c4, SWr1c5, SWr2c1, SWr2c2, SWr2c3, SWr2c4, SWr2c5, SWr3c1, SWr3c2, SWr3c3, SWr3c4, SWr3c5, SWr4c1, SWr4c2: footprint my syms-foots:ChocV1_duplex_hotswap_topor -> my syms-foots:Choc-and-KS33-Hotswap-Choc-1U
- moved REF** 1.94 mm to (156.3, 83.7)
- moved H1 0.46 mm to (145.0, 122.9)
Connections:
- SWr4c1 pad 2: GND2 -> db1
- SWr4c2 pad 2: GND2 -> db2
Routing:
- net GND2: track 75.1 -> 92.3 mm, vias 0 -> 4
- net r1c1: track 73.8 -> 59.6 mm, vias 2 -> 3
- net db2: track 59.7 -> 47.6 mm, vias 0 -> 2
- net r2c3: track 123.1 -> 111.8 mm, vias 2 -> 3
- net r2c4: track 116.6 -> 105.7 mm, vias 2 -> 3
- net r1c3: track 122.4 -> 112.2 mm, vias 2 -> 3
- net db1: track 40.3 -> 30.4 mm, vias 0 -> 1
- net r1c2: track 92.9 -> 83.6 mm, vias 2 -> 3
- net r1c4: track 142.8 -> 133.9 mm, vias 2 -> 3
- net r1c5: track 138.3 -> 129.6 mm, vias 2 -> 3
- net r2c5: track 128.0 -> 119.9 mm, vias 2 -> 3
- net r3c3: track 93.3 -> 86.2 mm, vias 2 -> 3
- net r2c1: track 51.5 -> 44.6 mm, vias 2 -> 3
- net r3c1: track 48.3 -> 42.4 mm, vias 2 -> 3
- net r2c2: track 74.9 -> 70.1 mm, vias 2 -> 3
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Other:
- outline, holes or cut-outs redrawn

Commit message: Add files via upload
Parts:
- added BT3: Breakaway Tabs, kbd_local:Breakaway_Tabs, F.Cu at (132.4, 116.1)
- moved BT3 0.50 mm to (160.9, 130.2)
- moved SWr4c1 0.50 mm to (150.7, 134.4)
- moved BT3 0.50 mm to (132.2, 116.6)
- moved H1 0.50 mm to (145.1, 123.4)
- moved REF** 0.50 mm to (160.7, 140.2)
- moved SWr4c2 0.50 mm to (133.0, 126.1)
Other:
- board size 129.8 x 98.6 mm -> 129.8 x 99.1 mm

Commit message: Add files via upload
Parts:
- removed J1: MJ-4PP-9, my syms-foots:TRRS-MJ-4PP-9_dual_topor
- added ?: , , F.Cu at (215.2, 91.5)
- added ?: , , F.Cu at (216.2, 79.1)
- added REF**: RTLECS MG03254 90 m, my syms-foots:RTLECS_MG03254_90_m, F.Cu at (215.7, 86.7)
- moved ? 1.56 mm to (216.0, 81.9)
Routing:
- net VCC: track 26.9 -> 19.8 mm
- net data: track 33.1 -> 31.3 mm
- net GND: track 58.9 -> 57.2 mm

Commit message: Add files via upload
Parts:
- moved REF** 1.46 mm to (207.5, 86.8)
Routing:
- net VCC: track 19.8 -> 22.3 mm
- net r1c1: track 59.6 -> 60.4 mm
- net r2c2: track 70.1 -> 70.9 mm
