File: ambra.kicad_sch (KiCad schematic)
At the start: 26 parts, among them J3 MTSW-103-07-S-S-225, J4 MTSW-103-07-S-S-225, J5 MJ-4PP-9, J6 B2B-ZR_LF__SN_, SW1 SW_SPDT, U1 ProMicro_r

Commit message: Add files via upload
Parts:
- removed C1: GCM32ER71E106KA42L, GCM32ER71E106KA42L:CAPC3225X270N, symbol GCM32ER71E106KA42L:GCM32ER71E106KA42L
- removed C2: C0603C104K8RACTU, C0603C104K8RACTU:CAPC1608X95N, symbol C0603C104K8RACTU:C0603C104K8RACTU
Connections:
- net r1c5: now also U1.7 (D4/4); no longer U1.8 (C6/5)
- net r2c1: now also U1.1 (D3/TX0); no longer U1.2 (D2/RX1)
- net r2c2: now also U1.2 (D2/RX1); no longer U1.6 (SCL/D0/3)
- net r2c3: now also U1.16 (15/B1); no longer U1.1 (D3/TX0)
- net r2c4: now also U1.6 (SCL/D0/3); no longer U1.7 (D4/4)
- net r3c1: now also U1.9 (D7/6); no longer U1.15 (14/B3)
- net r3c3: now also U1.8 (C6/5); no longer U1.9 (D7/6)
- net r3c5: now also U1.15 (14/B3); no longer U1.16 (15/B1)
- net at U1.B+ (BAT+): no longer SW1.2 (B)
- new net BAT+: SW1.2 (B)

Commit message: Add files via upload
Parts:
- removed J5: MJ-4PP-9, my syms-foots:TRRS-MJ-4PP-9_dual_topor, symbol enki_lib:MJ-4PP-9
- added J7: MTSW-103-07-S-S-225, my syms-foots:RTLECS_MG03254_f, symbol MTSW-103-07-S-S-225:MTSW-103-07-S-S-225
Connections:
- net GND: now also J7.01
- net VCC: now also J7.02
- net data: now also J7.03
Changed lines of the file:
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@@
 	(paper "A4")
 	(junction
-		(at 64.77 139.7)
-		(diameter 0)
-		(color 0 0 0 0)
-	)
-	(junction
 		(at 86.36 40.005)
 		(diameter 0)
@@
 	(wire
 		(pts
-			(xy 64.77 139.7) (xy 67.31 139.7)
-		)
-		(stroke
-			(width 0)
-			(type default)
-		)
-	)
-	(wire
-		(pts
 			(xy 167.005 33.655) (xy 167.005 37.465)
 		)
@@
 	(wire
 		(pts
-			(xy 131.445 33.655) (xy 131.445 37.465)
+			(xy 81.28 143.51) (xy 81.28 142.875)
 		)
 		(stroke
@@
 	(wire
 		(pts
-			(xy 246.38 44.45) (xy 246.38 48.26)
+			(xy 131.445 33.655) (xy 131.445 37.465)
 		)
 		(stroke
@@
 	(wire
 		(pts
-			(xy 196.85 123.19) (xy 198.12 123.19)
+			(xy 246.38 44.45) (xy 246.38 48.26)
 		)
 		(stroke
@@
 	(wire
 		(pts
-			(xy 64.77 139.7) (xy 64.77 140.97)
+			(xy 196.85 123.19) (xy 198.12 123.19)
 		)
 		(stroke
@@
 	(global_label "data"
 		(shape input)
-		(at 64.77 143.51 270)
+		(at 81.28 137.795 0)
 		(fields_autoplaced yes)
 		(effects
@@
 				(size 1 1)
 			)
-			(justify right)
+			(justify left)
 		)
 		(property "Intersheetrefs" "${INTERSHEET_REFS}"
-			(at 64.8325 148.6257 90)
+			(at 86.9161 137.795 0)
 			(effects
 				(font
 					(size 1 1)
 				)
-				(justify right)
+				(justify left)
 				(hide yes)
 			)
@@
 	(global_label "VCC"
 		(shape input)
-		(at 64.77 142.24 0)
+		(at 81.28 140.335 0)
 		(fields_autoplaced yes)
 		(effects
@@
 		)
 		(property "Intersheetrefs" "${INTERSHEET_REFS}"
-			(at 69.4571 142.1775 0)
+			(at 85.9671 140.2725 0)
 			(effects
 				(font
@@
 	)
 	(symbol
+		(lib_id "MTSW-103-07-S-S-225:MTSW-103-07-S-S-225")
+		(at 68.58 140.335 180)
+		(unit 1)
+		(exclude_from_sim no)
+		(in_bom yes)
+		(on_board yes)
+		(dnp no)
+		(fields_autoplaced yes)
+		(property "Reference" "J7"
+			(at 68.58 130.81 0)
+			(effects
+				(font
+					(size 1.27 1.27)
+				)
+			)
+		)
+		(property "Value" "MTSW-103-07-S-S-225"
+			(at 68.58 133.35 0)
+			(effects
+				(font
+					(size 1.27 1.27)
+				)
+			)
+		)
+		(property "Footprint" "my syms-foots:RTLECS_MG03254_f"
+			(at 68.58 140.335 0)
+			(effects
+				(font
+					(size 1.27 1.27)
+				)
+				(justify bottom)
+				(hide yes)
+			)
+		)
+		(property "Datasheet" ""
+			(at 68.58 140.335 0)
+			(effects
+				(font
+					(size 1.27 1.27)
+				)
+				(hide yes)
+			)
+		)
+		(property "Description" ""
+			(at 68.58 140.335 0)
+			(effects
+				(font
+					(size 1.27 1.27)
+				)
+				(hide yes)
+			)
+		)
+		(property "MF" "Samtec"
+			(at 68.58 140.335 0)
+			(effects
+				(font
+					(size 1.27 1.27)
+				)
+				(justify bottom)
+				(hide yes)
+			)
+		)
+		(property "Description_1" "\n                        \n                            HEADER, 3 CONTACTS, 1 ROW, THROUGH HOLE, 2.54 MM; Connector Systems:Board-to-Board; Pitch Spacing:2.54mm; No. of Rows:1Rows; No. of Contacts:3Contacts; Contact Termination Type:Through Hole; Product Range:MTSW Series; Gender:Header RoHS Compliant: Yes\n                        \n"
+			(at 68.58 140.335 0)
+			(effects
+				(font
+					(size 1.27 1.27)
+				)
+				(justify bottom)
+				(hide yes)
+			)
+		)
+		(property "Package" "None"
+			(at 68.58 140.335 0)
+			(effects
+				(font
+					(size 1.27 1.27)
+				)
+				(justify bottom)
+				(hide yes)
+			)
+		)
+		(property "Price" "None"
+			(at 68.58 140.335 0)
+			(effects
+				(font
+					(size 1.27 1.27)
+				)
+				(justify bottom)
+				(hide yes)
+			)
+		)
+		(property "Check_prices" "https://www.snapeda.com/parts/MTSW10307SS225/Samtec/view-part/?ref=eda"
+			(at 68.58 140.335 0)
+			(effects
+				(font
+					(size 1.27 1.27)
+				)
+				(justify bottom)
+				(hide yes)
+			)
+		)
+		(property "STANDARD" "Manufacturer Recommendations"
+			(at 68.58 140.335 0)
+			(effects
+				(font
+					(size 1.27 1.27)
+				)
+				(justify bottom)
+				(hide yes)
+			)
+		)
+		(property "PARTREV" "R"
+			(at 68.58 140.335 0)
+			(effects
+				(font
+					(size 1.27 1.27)
+				)
+				(justify bottom)
+				(hide yes)
+			)
+		)
+		(property "SnapEDA_Link" "https://www.snapeda.com/parts/MTSW10307SS225/Samtec/view-part/?ref=snap"
+			(at 68.58 140.335 0)
+			(effects
+				(font
+					(size 1.27 1.27)
+				)
+				(justify bottom)
+				(hide yes)
+			)
+		)
+		(property "MP" "MTSW10307SS225"
+			(at 68.58 140.335 0)
+			(effects
+				(font
+					(size 1.27 1.27)
+				)
+				(justify bottom)
+				(hide yes)
+			)
+		)
+		(property "Availability" "In Stock"
+			(at 68.58 140.335 0)
+			(effects
+				(font
+					(size 1.27 1.27)
+				)
+				(justify bottom)
+				(hide yes)
+			)
+		)
+		(property "MANUFACTURER" "Samtec"
+			(at 68.58 140.335 0)
+			(effects
+				(font
+					(size 1.27 1.27)
+				)
+				(justify bottom)
+				(hide yes)
+			)
+		)
+		(pin "02"
+		)
+		(pin "03"
+		)
+		(pin "01"
+		)
+		(instances
+			(project "ambra"
+				(path "/eaef1172-3351-417c-bfc4-74a598f141cb"
+					(reference "J7")
+					(unit 1)
+				)
+			)
+		)
+	)
+	(symbol
 		(lib_id "power:GND")
 		(at 217.805 67.945 0)
@@
 	)
 	(symbol
-		(lib_id "enki_lib:MJ-4PP-9")
-		(at 59.69 141.605 0)
-		(unit 1)
-		(exclude_from_sim no)
-		(in_bom yes)
-		(on_board yes)
-		(dnp no)
-		(property "Reference" "J5"
-			(at 60.4774 134.5946 0)
-			(effects
-				(font
-					(size 1.27 1.27)
-				)
-			)
-		)
-		(property "Value" "MJ-4PP-9"
-			(at 60.4774 136.906 0)
-			(effects
-				(font
-					(size 1.27 1.27)
-				)
-			)
-		)
-		(property "Footprint" "my syms-foots:TRRS-MJ-4PP-9_dual_topor"
-			(at 66.675 137.16 0)
-			(effects
-				(font
-					(size 1.27 1.27)
-				)
-				(hide yes)
-			)
-		)
-		(property "Datasheet" "~"
-			(at 66.675 137.16 0)
-			(effects
-				(font
-					(size 1.27 1.27)
-				)
-				(hide yes)
-			)
-		)
-		(property "Description" ""
-			(at 59.69 141.605 0)
-			(effects
-				(font
-					(size 1.27 1.27)
-				)
-				(hide yes)
-			)
-		)
-		(pin "R1"
-		)
-		(pin "R2"
-		)
-		(pin "S"
-		)
-		(pin "T"
-		)
-		(instances
-			(project "ambra"
-				(path "/eaef1172-3351-417c-bfc4-74a598f141cb"
-					(reference "J5")
-					(unit 1)
-				)
-			)
-		)
-	)
-	(symbol
 		(lib_id "enki_lib:SW_PUSH")
 		(at 156.845 52.705 0)
@@
 	(symbol
 		(lib_id "power:GND")
-		(at 67.31 139.7 90)
+		(at 81.28 143.51 90)
 		(unit 1)
 		(exclude_from_sim no)
@@
 		(fields_autoplaced yes)
 		(property "Reference" "#PWR03"
-			(at 73.66 139.7 0)
+			(at 87.63 143.51 0)
 			(effects
 				(font
@@
 		)
 		(property "Value" "GND"
-			(at 71.8725 139.7 0)
+			(at 85.8425 143.51 0)
 			(effects
 				(font
@@
 		)
 		(property "Footprint" ""
-			(at 67.31 139.7 0)
+			(at 81.28 143.51 0)
 			(effects
 				(font
@@
 		)
 		(property "Datasheet" ""
-			(at 67.31 139.7 0)
+			(at 81.28 143.51 0)
 			(effects
 				(font
@@
 		)
 		(property "Description" ""
-			(at 67.31 139.7 0)
+			(at 81.28 143.51 0)
 			(effects
 				(font
